File: UccMicroDuino/UccMicroDuino.kicad_pcb (KiCad board)
At the start: 2 copper layers, 8 parts, among them J1 Conn_01x10_Socket, J2 USB_A, U1 ATtiny85-20S

Commit message: Add files via upload
Parts:
- added D3: 3.6V 1/2mV, Diode_SMD:D_SOD-123, F.Cu at (110.3, 72.2)
- added D4: LED Green, ledSmd:ledSMD, F.Cu at (110.5, 77.0)
- added J1: USB_A, embeddedPcbUsb:USB_A_UCC, F.Cu at (130.7, 53.0)
- added R2: 68Ω 5% 1/8W, Resistor_SMD:R_0805_2012Metric_Pad1.20x1.40mm_HandSolder, F.Cu at (105.0, 72.0)
- added R3: 68Ω 5% 1/8W, Resistor_SMD:R_0805_2012Metric_Pad1.20x1.40mm_HandSolder, F.Cu at (105.0, 75.0)
- added R4: 330Ω 5% 1/8W, Resistor_SMD:R_0805_2012Metric_Pad1.20x1.40mm_HandSolder, F.Cu at (105.0, 78.0)
- added R5: 330Ω 5% 1/8W, Resistor_SMD:R_0805_2012Metric_Pad1.20x1.40mm_HandSolder, F.Cu at (105.0, 80.9)
- C1: value C -> 0.1u
- D1: value D_Filled -> PMLL4148L; footprint Diode_SMD:D_MiniMELF -> Diode_SMD:D_MELF_Handsoldering
- D2: value D_Zener -> 3.6V 1/2mV
- J2: renamed from J1; footprint Connector_PinHeader_2.54mm:PinHeader_1x10_P2.54mm_Vertical -> Connector_PinSocket_2.54mm:PinSocket_1x10_P2.54mm_Vertical
- R1: value R -> 1.5KΩ 5% 1/8W
- U1: value ATtiny85-20S -> ATtiny85-20SU
- renumbered D3 to D5
Connections:
- C1 pad 1: unconnected-(C1-Pad1) -> +5V
- C1 pad 2: unconnected-(C1-Pad2) -> GND
- D1 pad 2: unconnected-(D1-A-Pad2) -> Net-(D1-A)
- D2 pad 1: unconnected-(D2-K-Pad1) -> Net-(D2-K)
- D2 pad 2: unconnected-(D2-A-Pad2) -> GND
- D5 pad 1: unconnected-(D3-K-Pad1) -> Net-(D5-K)
- D5 pad 2: unconnected-(D3-A-Pad2) -> +5V
- J2 pad 1: unconnected-(J1-Pin_1-Pad1) -> +5V
- J2 pad 2: unconnected-(J1-Pin_2-Pad2) -> GND
- J2 pad 4: unconnected-(J1-Pin_4-Pad4) -> Net-(J2-Pin_4)
- J2 pad 5: unconnected-(J1-Pin_5-Pad5) -> Net-(D4-A)
- J2 pad 6: unconnected-(J1-Pin_6-Pad6) -> Net-(J2-Pin_6)
- J2 pad 7: unconnected-(J1-Pin_7-Pad7) -> Net-(J2-Pin_7)
- J2 pad 8: unconnected-(J1-Pin_8-Pad8) -> Net-(J2-Pin_8)
- J2 pad 9: unconnected-(J1-Pin_9-Pad9) -> Net-(J2-Pin_9)
- R1 pad 2: unconnected-(R1-Pad2) -> Net-(D2-K)
- U1 pad 1: unconnected-(U1-~{RESET}/PB5-Pad1) -> Net-(J2-Pin_9)
- U1 pad 2: unconnected-(U1-XTAL1/PB3-Pad2) -> Net-(J2-Pin_7)
- U1 pad 3: unconnected-(U1-XTAL2/PB4-Pad3) -> Net-(J2-Pin_8)
- U1 pad 4: unconnected-(U1-GND-Pad4) -> GND
- U1 pad 5: unconnected-(U1-AREF/PB0-Pad5) -> Net-(J2-Pin_4)
- U1 pad 6: unconnected-(U1-PB1-Pad6) -> Net-(D4-A)
- U1 pad 7: unconnected-(U1-PB2-Pad7) -> Net-(J2-Pin_6)
- U1 pad 8: unconnected-(U1-VCC-Pad8) -> +5V
Other:
- board outline added: 45 x 45 mm
