File: UccMicroDuino/UccMicroDuino.kicad_pcb (KiCad board)
At the start: 2 copper layers, 45 x 45 mm, 15 parts, among them J1 USB_A, J2 Conn_01x10_Socket, J2 USB_A, U1 ATtiny85-20SU

Commit message: Add files via upload
Parts:
- moved R5 58.6 mm to (162.0, 67.5), turned to 90 degrees
- moved R4 58.4 mm to (161.5, 63.0), turned to 90 degrees
- moved D4 57.3 mm to (165.8, 62.1), turned to 90 degrees
- moved R3 53.4 mm to (157.0, 63.0), turned to -90 degrees
- moved R2 49.3 mm to (153.5, 63.0), turned to -90 degrees
- moved D3 46.9 mm to (157.0, 68.2), turned to 90 degrees
- moved J2 39.2 mm to (153.8, 93.5), turned to 90 degrees
- moved D5 35.9 mm to (165.5, 68.4), turned to -90 degrees
- moved D2 33.3 mm to (153.5, 67.8), turned to 90 degrees
- moved U1 29.8 mm to (161.3, 84.5)
- moved D1 29.6 mm to (150.5, 66.4), turned to 90 degrees
- moved C1 26.4 mm to (164.5, 72.5), turned to 180 degrees
- moved J1 23.5 mm to (154.0, 56.0), turned to -90 degrees
- moved R1 13.6 mm to (151.5, 74.5)
- moved J2 5.91 mm to (126.7, 69.5)

Commit message: Add files via upload
Parts:
- moved J2 20.7 mm to (174.5, 93.5), turned to -90 degrees
- moved R2 10.9 mm to (156.5, 73.5)
- moved D2 4.65 mm to (157.8, 69.5), turned to 0 degrees
- moved D3 2.23 mm to (158.5, 66.5), turned to 0 degrees
- moved R1 1.58 mm to (153.0, 75.0)
Routing:
- net +5V: track 0.00 -> 52.9 mm
- net GND: track 0.00 -> 40.1 mm
- net Net-(D2-K): track 0.00 -> 26.5 mm
- net Net-(D4-A): track 0.00 -> 26.1 mm
- net Net-(J2-Pin_8): track 0.00 -> 23.3 mm
- net Net-(D3-K): track 0.00 -> 11.9 mm
- net Net-(J2-Pin_7): track 0.00 -> 10.7 mm
- net Net-(D1-A): track 0.00 -> 7.20 mm
- net Net-(D4-K): track 0.00 -> 4.34 mm
- net Net-(D5-K): track 0.00 -> 3.55 mm

Commit message: Add files via upload
Parts:
- moved R3 50.5 mm to (204.5, 80.0), turned to 0 degrees
- moved R1 49.2 mm to (201.0, 64.0), turned to 90 degrees
- moved R2 42.0 mm to (198.5, 72.0), turned to 180 degrees
- moved D3 39.1 mm to (196.5, 75.5), turned to 180 degrees
- moved D1 35.6 mm to (186.0, 68.4), turned to -90 degrees
- moved D2 33.4 mm to (190.5, 76.5)
- moved C1 29.4 mm to (193.0, 79.5), turned to -90 degrees
- moved J2 28.9 mm to (163.5, 66.8), turned to 0 degrees
- moved D4 20.5 mm to (155.7, 79.9), turned to -90 degrees
- moved U1 19.6 mm to (179.9, 78.2), turned to 90 degrees
- moved R4 12.1 mm to (155.5, 73.5)
- moved R5 6.80 mm to (155.5, 65.5)
- moved D5 6.70 mm to (171.7, 65.9)
- moved J1 0.70 mm to (154.0, 56.7)
Routing:
- net GND: track 40.1 -> 146.3 mm
- net Net-(D3-K): track 11.9 -> 78.5 mm
- net Net-(D2-K): track 26.5 -> 76.5 mm
- net Net-(D1-A): track 7.20 -> 46.2 mm
- net Net-(J2-Pin_8): track 23.3 -> 57.7 mm
- net Net-(J2-Pin_7): track 10.7 -> 41.4 mm
- net +5V: track 52.9 -> 80.2 mm
- net Net-(J2-Pin_4): track 0.00 -> 21.8 mm
- net Net-(J2-Pin_6): track 0.00 -> 19.5 mm
- net Net-(J2-Pin_9): track 0.00 -> 16.7 mm
- net Net-(D5-K): track 3.55 -> 16.4 mm
- net Net-(D4-A): track 26.1 -> 30.2 mm
- net Net-(D4-K): track 4.34 -> 3.71 mm
Other:
- board size 45 x 45 mm -> 63 x 45 mm

Commit message: Add files via upload
Parts:
- moved C1 21.0 mm to (174.5, 69.5), turned to 180 degrees
- moved R3 15.0 mm to (200.5, 65.5)
- moved R1 13.0 mm to (194.0, 75.0)
- moved D2 10.5 mm to (191.0, 66.0)
- moved D3 10.4 mm to (206.5, 78.5)
- moved R2 8.06 mm to (190.5, 71.0)
- moved D1 4.66 mm to (182.0, 66.0), turned to 180 degrees
Routing:
- net GND: track 146.3 -> 199.2 mm
- net +5V: track 80.2 -> 57.0 mm
- net Net-(D1-A): track 46.2 -> 33.8 mm
- net Net-(J2-Pin_7): track 41.4 -> 32.2 mm
- net Net-(J2-Pin_8): track 57.7 -> 63.0 mm
- net Net-(D2-K): track 76.5 -> 72.3 mm
- net Net-(D3-K): track 78.5 -> 77.3 mm

Commit message: Add files via upload
Parts:
- moved C1 1.47 mm to (174.7, 71.0)
- moved D1 1.47 mm to (182.2, 67.5)
- moved D2 1.47 mm to (191.2, 67.5)
- moved D3 1.47 mm to (206.7, 80.0)
- moved D4 1.47 mm to (155.9, 81.4)
- moved D5 1.47 mm to (171.9, 67.4)
- moved J2 1.47 mm to (163.7, 68.3)
- moved R1 1.47 mm to (194.2, 76.5)
- moved R2 1.47 mm to (190.7, 72.5)
- moved R3 1.47 mm to (200.7, 67.0)
- moved R4 1.47 mm to (155.7, 75.0)
- moved R5 1.47 mm to (155.7, 67.0)
- moved U1 1.47 mm to (180.1, 79.6)
- moved J1 0.70 mm to (154.0, 56.0)
Routing:
- net GND: track 199.2 -> 307.3 mm
- net Net-(D3-K): track 77.3 -> 74.1 mm
- net Net-(D1-A): track 33.8 -> 36.0 mm
- net Net-(D2-K): track 72.3 -> 73.8 mm
- net unconnected-(J2-Pin_10-Pad10): track 0.00 -> 0.58 mm
Other:
- board size 63 x 45 mm -> 62.5 x 45 mm
