File: UccMicroDuino/UccMicroDuino.kicad_sch (KiCad schematic)
At the start: 13 parts, among them J1 Pcb USB Type A, J2 Conn_01x10_Socket, U2 ATtiny85-20SU

Commit message: Add files via upload
Plano actualizado 14-04
Parts:
- renumbered D3 to D5, R3 to R2, R2 to R3
Changed lines of the file:
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@@
 		(dnp no)
 		(fields_autoplaced yes)
-		(property "Reference" "D3"
+		(property "Reference" "D5"
 			(at 260.35 82.2325 90)
 			(effects
@@
 			(project "UccMicroDuino"
 				(path "/f2c20679-f28d-47ad-9191-2bfbde129570"
-					(reference "D3")
+					(reference "D5")
 					(unit 1)
 				)
@@
 		(dnp no)
 		(fields_autoplaced yes)
-		(property "Reference" "#PWR05"
+		(property "Reference" "#PWR03"
 			(at 88.9 127 0)
 			(effects
@@
 			(project "UccMicroDuino"
 				(path "/f2c20679-f28d-47ad-9191-2bfbde129570"
-					(reference "#PWR05")
+					(reference "#PWR03")
 					(unit 1)
 				)
@@
 			(project "UccMicroDuino"
 				(path "/f2c20679-f28d-47ad-9191-2bfbde129570"
-					(reference "J1")
+					(reference "J2")
 					(unit 1)
 				)
@@
 		(on_board yes)
 		(dnp no)
-		(property "Reference" "#PWR09"
+		(property "Reference" "#PWR05"
 			(at 148.59 63.5 0)
 			(effects
@@
 			(project "UccMicroDuino"
 				(path "/f2c20679-f28d-47ad-9191-2bfbde129570"
-					(reference "#PWR09")
+					(reference "#PWR05")
 					(unit 1)
 				)
@@
 			(project "UccMicroDuino"
 				(path "/f2c20679-f28d-47ad-9191-2bfbde129570"
-					(reference "#PWR02")
+					(reference "#PWR09")
 					(unit 1)
 				)
@@
 		(dnp no)
 		(fields_autoplaced yes)
-		(property "Reference" "#PWR04"
+		(property "Reference" "#PWR01"
 			(at 57.15 118.11 0)
 			(effects
@@
 			(project "UccMicroDuino"
 				(path "/f2c20679-f28d-47ad-9191-2bfbde129570"
-					(reference "#PWR04")
+					(reference "#PWR01")
 					(unit 1)
 				)
@@
 		(dnp no)
 		(fields_autoplaced yes)
-		(property "Reference" "#PWR07"
+		(property "Reference" "#PWR06"
 			(at 173.99 104.14 0)
 			(effects
@@
 			(project "UccMicroDuino"
 				(path "/f2c20679-f28d-47ad-9191-2bfbde129570"
-					(reference "#PWR07")
+					(reference "#PWR06")
 					(unit 1)
 				)
@@
 		(dnp no)
 		(fields_autoplaced yes)
-		(property "Reference" "#PWR03"
+		(property "Reference" "#PWR07"
 			(at 173.99 142.24 0)
 			(effects
@@
 			(project "UccMicroDuino"
 				(path "/f2c20679-f28d-47ad-9191-2bfbde129570"
-					(reference "#PWR03")
+					(reference "#PWR07")
 					(unit 1)
 				)
@@
 			(project "UccMicroDuino"
 				(path "/f2c20679-f28d-47ad-9191-2bfbde129570"
-					(reference "#PWR01")
+					(reference "#PWR02")
 					(unit 1)
 				)
@@
 		(dnp no)
 		(fields_autoplaced yes)
-		(property "Reference" "#PWR06"
+		(property "Reference" "#PWR08"
 			(at 185.42 88.9 0)
 			(effects
@@
 			(project "UccMicroDuino"
 				(path "/f2c20679-f28d-47ad-9191-2bfbde129570"
-					(reference "#PWR06")
+					(reference "#PWR08")
 					(unit 1)
 				)
@@
 		(on_board yes)
 		(dnp no)
-		(property "Reference" "R3"
+		(property "Reference" "R2"
 			(at 107.95 104.14 90)
 			(effects
@@
 			(project "UccMicroDuino"
 				(path "/f2c20679-f28d-47ad-9191-2bfbde129570"
-					(reference "R3")
+					(reference "R2")
 					(unit 1)
 				)
@@
 		(on_board yes)
 		(dnp no)
-		(property "Reference" "R2"
+		(property "Reference" "R3"
 			(at 116.84 101.6 90)
 			(effects
@@
 			(project "UccMicroDuino"
 				(path "/f2c20679-f28d-47ad-9191-2bfbde129570"
-					(reference "R2")
+					(reference "R3")
 					(unit 1)
 				)
@@
 		(dnp no)
 		(fields_autoplaced yes)
-		(property "Reference" "#PWR08"
+		(property "Reference" "#PWR04"
 			(at 146.05 76.2 0)
 			(effects
@@
 			(project "UccMicroDuino"
 				(path "/f2c20679-f28d-47ad-9191-2bfbde129570"
-					(reference "#PWR08")
-					(unit 1)
-				)
+					(reference "#PWR04")
+					(unit 1)
+				)

Commit message: Add files via upload
Parts:
- removed J1: Pcb USB Type A, embeddedPcbUsb:USB_A_UCC, symbol Connector:USB_A
- added J1: USB_A, symbol usbLibrary:USB_A
- added R5: 330Ω 5% 1/8W, Resistor_SMD:R_0805_2012Metric_Pad1.20x1.40mm_HandSolder, symbol Device:R
- C1: value C -> 0.1u
- D5: footprint Diode_SMD:D_MiniMELF -> Diode_SMD:D_MELF_Handsoldering
- J2: footprint Connector_PinHeader_2.54mm:PinHeader_1x10_P2.54mm_Vertical -> Connector_PinSocket_2.54mm:PinSocket_1x10_P2.54mm_Vertical
Connections:
- net +5V: now also C1.1, D5.2 (A)
- net GND: now also C1.2, J1.4 (GND), R5.1
- net at D5.1 (K): now also R5.2
- net at D3.1 (K), R3.1: now also J1.3 (D+)
- net at D1.1 (K), R1.2, R2.1: now also J1.2 (D-)
- net 1: no longer names the net of D5.2 (A)
- net 1: now also J1.1 (VBUS)
Other:
- note added: "DC Power"
- note added: "Power Led"
- moved on the sheet: D5

Commit message: Add files via upload
Parts:
- J1: footprint (none) -> embeddedPcbUsb:USB_A_UCC
Changed lines of the file:
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@@
 			)
 		)
-		(property "Footprint" ""
+		(property "Footprint" "embeddedPcbUsb:USB_A_UCC"
 			(at 60.96 102.87 0)
 			(effects
